Commit message: 200331

File: fingertest/urdf/fingertest.urdf.xacro (robot description, xacro)
@@ -13,5 +13,5 @@
         rpy="0 0 0" />
       <mass
-        value="0.0027" />
+        value="0.027" />
       <inertia
         ixx="0"
@@ -53,5 +53,5 @@
         rpy="0 0 0" />
       <mass
-        value="0.002" />
+        value="0.02" />
       <inertia
         ixx="0"
@@ -76,9 +76,9 @@
       </material>
     </visual>
-    <collision name="${side}_Link1_bumper">
-      <origin
-        xyz="0 0 0"
-        rpy="0 0 0" />
-      <geometry name="${side}_Link1_bumper">
+    <collision>
+      <origin
+        xyz="0 0 0"
+        rpy="0 0 0" />
+      <geometry>
         <mesh
           filename="package://fingertest/meshes/Link_1.STL" />
@@ -116,5 +116,5 @@
         rpy="0 0 0" />
       <mass
-        value="0.00197" />
+        value="0.0197910341256244" />
       <inertia
         ixx="0"
@@ -139,9 +139,9 @@
       </material>
     </visual>
-    <collision name="${side}_Link2_bumper">
-      <origin
-        xyz="0 0 0"
-        rpy="0 0 0" />
-      <geometry name="${side}_Link2_bumper">
+    <collision>
+      <origin
+        xyz="0 0 0"
+        rpy="0 0 0" />
+      <geometry>
         <mesh
           filename="package://fingertest/meshes/Link_2.STL" />
@@ -169,5 +169,5 @@
         rpy="0 0 0" />
       <mass
-        value="0.0027" />
+        value="0.027" />
       <inertia
         ixx="0"
@@ -192,9 +192,9 @@
       </material>
     </visual>
-    <collision name="${side}_Link3_bumper">
-      <origin
-        xyz="0 0 0"
-        rpy="0 0 0" />
-      <geometry name="${side}_Link3_bumper">
+    <collision name="bumper_${side}_collision">
+      <origin
+        xyz="0 0 0"
+        rpy="0 0 0" />
+      <geometry name="bumper_${side}_collision">
         <mesh
           filename="package://fingertest/meshes/Link_3.STL" />
@@ -246,16 +246,16 @@
   </transmission>
   <xacro:fingertest_gazebo side="${side}"/>
-  <gazebo reference="${side}_Link_1">
-   <sensor name="${side}_Link_1_sensor" type="contact">
+  <gazebo reference="${side}_Link_3">
+   <sensor name="${side}_Link_3_sensor" type="contact">
         <visualize>true</visualize>
         <always_on>true</always_on>
         <update_rate>50.0</update_rate>
         <contact>
-            <collision>${side}_Link_1_fixed_joint_lump__${side}_Link1_bumper_collision</collision>
+            <collision>bumper_${side}_collision_collison</collision>
         </contact>
         <plugin name="gazebo_ros_bumper_controller" filename="libgazebo_ros_bumper.so">
                 <alwaysOn>true</alwaysOn>
                 <updateRate>10.0</updateRate>
-                <bumperTopicName>${side}_Link1_bumper</bumperTopicName>
+                <bumperTopicName>${side}_bumper_finger</bumperTopicName>
                 <frameName>world</frameName>
             </plugin>
@@ -265,44 +265,5 @@
     <mu2>0.1</mu2>
     <gravity>true</gravity>
-    </gazebo>
-    <gazebo reference="${side}_Link_2">
-   <sensor name="${side}_Link_2_sensor" type="contact">
-        <visualize>true</visualize>
-        <always_on>true</always_on>
-        <update_rate>50.0</update_rate>
-        <contact>
-            <collision>${side}_Link_2_fixed_joint_lump__${side}_Link2_bumper_collision</collision>
-        </contact>
-        <plugin name="gazebo_ros_bumper_controller" filename="libgazebo_ros_bumper.so">
-                <alwaysOn>true</alwaysOn>
-                <updateRate>10.0</updateRate>
-                <bumperTopicName>${side}_Link2_bumper</bumperTopicName>
-                <frameName>world</frameName>
-            </plugin>
-    </sensor>
-    <material>Gazebo/Red</material>
-    <mu1>0.1</mu1>
-    <mu2>0.1</mu2>
-    <gravity>true</gravity>
-    </gazebo>
-  <gazebo reference="${side}_Link_3">
-   <sensor name="${side}_Link_3_sensor" type="contact">
-        <visualize>true</visualize>
-        <always_on>true</always_on>
-        <update_rate>50.0</update_rate>
-        <contact>
-            <collision>${side}_Link_3_fixed_joint_lump__${side}_Link3_bumper_collision</collision>
-        </contact>
-        <plugin name="gazebo_ros_bumper_controller" filename="libgazebo_ros_bumper.so">
-                <alwaysOn>true</alwaysOn>
-                <updateRate>10.0</updateRate>
-                <bumperTopicName>${side}_Link3_bumper</bumperTopicName>
-                <frameName>world</frameName>
-            </plugin>
-    </sensor>
-    <material>Gazebo/Red</material>
-    <mu1>0.1</mu1>
-    <mu2>0.1</mu2>
-    <gravity>true</gravity>
+    <selfCollide>false</selfCollide>
 </gazebo>
   <!-- <gazebo reference="bumper_finger">

File: gripper_base/urdf/gripper_base.xacro (robot description, xacro)
@@ -109,4 +109,5 @@
     <axis
       xyz="0 0 -1" />
+    <limit effort="60" velocity="100000" lower="0" upper="3.14" />
   </joint>
   <link
@@ -164,4 +165,5 @@
     <axis
       xyz="0 0 1" />
+    <limit effort="60" velocity="10000" lower="0" upper="3.14" />
   </joint>
   <transmission name="tran1">
