Commit message: 200401

File: fingertest/urdf/fingertest.xacro (robot description, xacro)
@@ -261,7 +261,4 @@
             </plugin>
     </sensor>
-    <material>Gazebo/Red</material>
-    <mu1>0.1</mu1>
-    <mu2>0.1</mu2>
     <gravity>true</gravity>
     </gazebo>
@@ -281,7 +278,4 @@
             </plugin>
     </sensor>
-    <material>Gazebo/Red</material>
-    <mu1>0.1</mu1>
-    <mu2>0.1</mu2>
     <gravity>true</gravity>
     </gazebo>
@@ -301,7 +295,4 @@
             </plugin>
     </sensor>
-    <material>Gazebo/Red</material>
-    <mu1>0.1</mu1>
-    <mu2>0.1</mu2>
     <gravity>true</gravity>
 </gazebo>

File: gripper/urdf/3fgripper.xacro (robot description, xacro)
@@ -6,5 +6,5 @@
     <link name="world"/>
   <xacro:gripper_base parent="world" child="gripper_base_link">
-    <origin xyz="0 0 0" rpy="0 0 0"  />
+    <origin xyz="0 0 0.22" rpy="3.14 0 0"  />
   </xacro:gripper_base>
   <xacro:fingertest side="r" parent="r_finger_link" child="r_base_link">
